File: power.kicad_sch (KiCad schematic)
At the start: 68 parts, among them U1 LFE5U-85F-6BG381C, U5 TLV62569DBV, U6 TLV62569DBV, U7 TLV62569DBV, U8 TLV62569DBV

Commit message: Adding BOM - adding DNP to some components
Parts:
- 1.1V_1, RP1, RP2, RP3, RP4, RV2: now not fitted
Changed lines of the file:
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@@
 		(in_bom yes)
 		(on_board yes)
-		(dnp no)
+		(dnp yes)
 		(property "Reference" "RP1"
 			(at 271.78 76.708 0)
@@
 		(in_bom yes)
 		(on_board yes)
-		(dnp no)
+		(dnp yes)
 		(property "Reference" "RP2"
 			(at 271.78 107.188 0)
@@
 		(in_bom yes)
 		(on_board yes)
-		(dnp no)
+		(dnp yes)
 		(property "Reference" "RP3"
 			(at 271.78 137.668 0)
@@
 		(in_bom yes)
 		(on_board yes)
-		(dnp no)
+		(dnp yes)
 		(property "Reference" "RV2"
 			(at 19.685 33.02 0)
@@
 		(in_bom yes)
 		(on_board yes)
-		(dnp no)
+		(dnp yes)
 		(property "Reference" "RP4"
 			(at 163.83 163.703 0)
@@
 		(in_bom yes)
 		(on_board yes)
-		(dnp no)
+		(dnp yes)
 		(property "Reference" "1.1V_1"
 			(at 23.4442 50.2666 0)
